Commit message: finish one simple example of talos

File: Robots/talos/talos_reduced_armfixed_floatingbase.urdf (robot description, URDF)
Before this commit: robot talos, 60 links, 59 joints
Links:
- added link Px, mass 0
- added link Py, mass 0
- added link Pz, mass 0
- added link Rx, mass 0
- added link Ry, mass 0
- added link ground, mass 0
Joints:
- added joint Px: type prismatic, parent ground, child Px, origin xyz=0 0 0, axis 1 0 0, limit lower=-2 upper=2 effort=1000 velocity=1000
- added joint Py: type prismatic, parent Px, child Py, origin xyz=0 0 0, axis 0 1 0, limit lower=-2 upper=2 effort=1000 velocity=1000
- added joint Pz: type prismatic, parent Py, child Pz, origin xyz=0 0 0, axis 0 0 1, limit lower=-2 upper=2 effort=1000 velocity=1000
- added joint Rx: type revolute, parent Pz, child Rx, origin xyz=0 0 0, axis 1 0 0, limit lower=-1000 upper=1000 effort=1000 velocity=1000
- added joint Ry: type revolute, parent Rx, child Ry, origin xyz=0 0 0, axis 0 1 0, limit lower=-1000 upper=1000 effort=1000 velocity=1000
- added joint Rz: type revolute, parent Ry, child base_link, origin xyz=0 0 0, axis 0 0 1, limit lower=-1000 upper=1000 effort=1000 velocity=1000
