Commit message: clean up Digit code

File: Robots/digit-v3/digit-v3-floatingbase-springfixed.urdf (robot description, URDF)
Before this commit: robot digit-v3-modified, 33 links, 32 joints
Links:
- added link left_A2, mass 0.090983; collision sphere radius=0.0; visual sphere radius=0.0
- added link left_B2, mass 0.079507; collision sphere radius=0.0; visual sphere radius=0.0
- added link left_ach2, mass 0.178148; collision sphere radius=0.0; visual sphere radius=0.0
- added link left_achilles_rod, mass 0.; collision mesh filename=meshes/leg-v3/achilles-rod.stl; visual mesh filename=meshes/leg-v3/achilles-rod.stl
- added link left_toe_A, mass 0.139557; collision mesh filename=meshes/leg-v3/toe-output.stl; visual mesh filename=meshes/leg-v3/toe-output.stl
- added link left_toe_A_rod, mass 0.; collision mesh filename=meshes/leg-v3/toe-a-rod.stl; visual mesh filename=meshes/leg-v3/toe-a-rod.stl
- added link left_toe_B, mass 0.139557; collision mesh filename=meshes/leg-v3/toe-output.stl; visual mesh filename=meshes/leg-v3/toe-output.stl
- added link left_toe_B_rod, mass 0.; collision mesh filename=meshes/leg-v3/toe-b-rod.stl; visual mesh filename=meshes/leg-v3/toe-b-rod.stl
- added link right_A2, mass 0.090983; collision sphere radius=0.0; visual sphere radius=0.0
- added link right_B2, mass 0.079507; collision sphere radius=0.0; visual sphere radius=0.0
- added link right_ach2, mass 0.178148; collision sphere radius=0.0; visual sphere radius=0.0
- added link right_achilles_rod, mass 0.; collision mesh filename=meshes/leg-v3/achilles-rod.stl scale=1 1 1; visual mesh filename=meshes/leg-v3/achilles-rod.stl scale=1 1 1
- added link right_toe_A, mass 0.139557; collision mesh filename=meshes/leg-v3/toe-output.stl scale=1 1 1; visual mesh filename=meshes/leg-v3/toe-output.stl scale=1 1 1
- added link right_toe_A_rod, mass 0.; collision mesh filename=meshes/leg-v3/toe-a-rod.stl scale=1 1 1; visual mesh filename=meshes/leg-v3/toe-a-rod.stl scale=1 1 1
- added link right_toe_B, mass 0.139557; collision mesh filename=meshes/leg-v3/toe-output.stl scale=1 1 1; visual mesh filename=meshes/leg-v3/toe-output.stl scale=1 1 1
- added link right_toe_B_rod, mass 0.; collision mesh filename=meshes/leg-v3/toe-b-rod.stl scale=1 1 1; visual mesh filename=meshes/leg-v3/toe-b-rod.stl scale=1 1 1
Joints:
- added joint left_A2: type revolute, parent left_toe_A_rod, child left_A2, origin xyz=0 0 0 rpy=0 0 0, axis 0 1 0, limit lower=-1.7453 upper=1.7453 effort=0.9 velocity=11.5
- added joint left_B2: type revolute, parent left_toe_B_rod, child left_B2, origin xyz=0 0 0 rpy=0 0 0, axis 0 1 0, limit lower=-1.7453 upper=1.7453 effort=0.9 velocity=11.5
- added joint left_ach2: type revolute, parent left_achilles_rod, child left_ach2, origin xyz=0 0 0 rpy=0 0 0, axis 0 1 0, limit lower=-1.7453 upper=1.7453 effort=0.9 velocity=11.5
- added joint left_achilles_rod: type revolute, parent left_hip_pitch, child left_achilles_rod, origin xyz=0 0 0.046 rpy=0.0087528908613780896652567520277444 0.07085157762907765000015558598534 -1.4355410054288866295024718056084, axis 0 0 1, limit lower=-1.7453 upper=1.7453 effort=12.5 velocity=8.5085
- added joint left_toe_A: type revolute, parent left_tarsus, child left_toe_A, origin xyz=0.059 -0.034 -0.0276 rpy=3.1415926535897932384626433832795 0 -1.5526449025733231046331184188602, axis 0 0 1, limit lower=-0.8077 upper=0.7851 effort=0.9 velocity=11.5
- added joint left_toe_A_rod: type revolute, parent left_toe_A, child left_toe_A_rod, origin xyz=0.057 0 -0.008 rpy=-0.037175987474526640819139089444434 0.0069420091856212517295032782271846 -1.5437619437662688515189302052022, axis 0 0 1, limit lower=-1.7453 upper=1.7453 effort=0.9 velocity=11.5
- added joint left_toe_B: type revolute, parent left_tarsus, child left_toe_B, origin xyz=0.111 -0.034 0.0276 rpy=0         0   -1.5526446425200970402613620535703, axis 0 0 1, limit lower=-0.8010 upper=0.7950 effort=0.9 velocity=11.5
- added joint left_toe_B_rod: type revolute, parent left_toe_B, child left_toe_B_rod, origin xyz=0.057 0 -0.008 rpy=-0.053844685552438438513878082858355 0.0022826832958013874852465363574083 1.5418663490001245364169335516635, axis 0 0 1, limit lower=-1.7453 upper=1.7453 effort=0.9 velocity=11.5
- added joint right_A2: type revolute, parent right_toe_A_rod, child right_A2, origin xyz=0 0 0 rpy=0 0 0, axis 0 1 0, limit lower=-1.7453 upper=1.7453 effort=0.9 velocity=11.5
- added joint right_B2: type revolute, parent right_toe_B_rod, child right_B2, origin xyz=0 0 0 rpy=0 0 0, axis 0 1 0, limit lower=-1.7453 upper=1.7453 effort=0.9 velocity=11.5
- added joint right_ach2: type revolute, parent right_achilles_rod, child right_ach2, origin xyz=0 0 0 rpy=0 0 0, axis 0 1 0, limit lower=-1.7453 upper=1.7453 effort=0.9 velocity=11.5
- added joint right_achilles_rod: type revolute, parent right_hip_pitch, child right_achilles_rod, origin xyz=0 0 0.046 rpy=-0.0087523017375784415566863927438135 0.070851391807226243857442682383407 1.4355417226017064269427692124736, axis 0 0 1, limit lower=-1.7453 upper=1.7453 effort=12.5 velocity=8.5085
- added joint right_toe_A: type revolute, parent right_tarsus, child right_toe_A, origin xyz=0.059 0.034 -0.0276 rpy=3.1415926535897932384626433832795 0 1.5526446425200970402613620535703, axis 0 0 1, limit lower=-0.7851 upper=0.8077 effort=0.9 velocity=11.5
- added joint right_toe_A_rod: type revolute, parent right_toe_A, child right_toe_A_rod, origin xyz=0.057 0 -0.008 rpy=0.03717647899635967423392912678537 0.0069418384185932916277672610760874 1.5437611240201540852012840332463, axis 0 0 1, limit lower=-1.7453 upper=1.7453 effort=0.9 velocity=11.5
- added joint right_toe_B: type revolute, parent right_tarsus, child right_toe_B, origin xyz=0.111 0.034 0.0276 rpy=0         0    1.5526446425200970402613620535703, axis 0 0 1, limit lower=-0.7950 upper=0.8010 effort=0.9 velocity=11.5
- added joint right_toe_B_rod: type revolute, parent right_toe_B, child right_toe_B_rod, origin xyz=0.057 0 -0.008 rpy=0.053844685552438438513878082858355 0.0022826832958013874852465363574083 -1.5418663490001245364169335516635, axis 0 0 1, limit lower=-1.7453 upper=1.7453 effort=0.9 velocity=11.5
- joint left_elbow: origin xyz=0 -0.0385 0.185 rpy=1.5707963267948966192313216916398 -0.3926991 0 -> xyz=0 -0.0385 0.185 rpy=1.57079632679489661923 -0.3926991 0; type fixed -> continuous
- joint left_shoulder_pitch: origin xyz=-0.00317 -0.011055 0.0555 rpy=1.5707963267948966192313216916398 1.875658163397448285891755404009 -0.2792527 -> xyz=-0.00317 -0.011055 0.0555 rpy=1.57079632679489661923 0.785398163397 -0.2792527; type fixed -> continuous
- joint left_shoulder_roll: origin xyz=-0.001 0.12 0.4 rpy=-1.5707963267948966192313216916398 -1.5467303 1.5707963267948966192313216916398 -> xyz=-0.001 0.12 0.4 rpy=-1.57079632679489661923 -1.3962633 1.57079632679489661923; type fixed -> continuous
- joint left_shoulder_yaw: origin xyz=0 -0.165 -0.1 rpy=1.5707963267948966192313216916398 -0.14981736 0 -> xyz=0 -0.165 -0.1 rpy=1.57079632679489661923 0 0; type fixed -> continuous
- joint right_elbow: type fixed -> continuous
- joint right_shoulder_pitch: origin xyz=-0.00317 0.011055 0.0555 rpy=-1.5707963267948966192313216916398 1.875658163397448285891755404009 0.2792527 -> xyz=-0.00317 0.011055 0.0555 rpy=-1.5707963267948966192313216916398 0.78539816339744830961566084581988 0.2792527; type fixed -> continuous
- joint right_shoulder_roll: origin xyz=-0.001 -0.12 0.4 rpy=1.5707963267948966192313216916398 -1.5467303 -1.5707963267948966192313216916398 -> xyz=-0.001 -0.12 0.4 rpy=1.5707963267948966192313216916398 -1.3962633 -1.5707963267948966192313216916398; type fixed -> continuous
- joint right_shoulder_yaw: origin xyz=0 0.165 -0.1 rpy=-1.5707963267948966192313216916398 -0.14981736 0 -> xyz=0 0.165 -0.1 rpy=-1.5707963267948966192313216916398         0         0; type fixed -> continuous

Commit message: hotfix: digit urdf arm

File: Robots/digit-v3/digit-v3-floatingbase-springfixed.urdf (robot description, URDF)
Before this commit: robot digit-v3-floatingbase-springfixed, 49 links, 48 joints
Joints:
- joint left_elbow: type continuous -> revolute
- joint left_shoulder_pitch: type continuous -> revolute
- joint left_shoulder_roll: type continuous -> revolute
- joint left_shoulder_yaw: type continuous -> revolute
- joint right_elbow: type continuous -> revolute
- joint right_shoulder_pitch: type continuous -> revolute
- joint right_shoulder_roll: type continuous -> revolute
- joint right_shoulder_yaw: type continuous -> revolute
