Commit message: update Kinova Waitr planner and its nanobind

File: Robots/kinova-gen3/kinova_grasp.urdf (robot description, URDF)
Before this commit: robot gen3_robotiq_2f_85, 11 links, 10 joints
Links:
- link base: geometry collision mesh filename=meshes/base_link.STL; visual mesh filename=meshes/base_link.STL
- link bracelet_link: geometry collision mesh filename=meshes/bracelet_with_vision_link.STL; visual mesh filename=meshes/bracelet_with_vision_link.STL
- link cube_link: geometry collision mesh filename=meshes/cube_all_corners_shifted_scaled_origin_v2.STL; visual mesh filename=meshes/cube_all_corners_shifted_scaled_origin_v2.STL
- link forearm_link: geometry collision mesh filename=meshes/forearm_link.STL; visual mesh filename=meshes/forearm_link.STL
- link gripper_base: geometry collision mesh filename=meshes/base_of_gripper.STL; visual mesh filename=meshes/base_of_gripper.STL
- link half_arm_1_link: geometry collision mesh filename=meshes/half_arm_1_link.STL; visual mesh filename=meshes/half_arm_1_link.STL
- link half_arm_2_link: geometry collision mesh filename=meshes/half_arm_2_link.STL; visual mesh filename=meshes/half_arm_2_link.STL
- link shoulder_link: geometry collision mesh filename=meshes/shoulder_link.STL; visual mesh filename=meshes/shoulder_link.STL
- link spherical_wrist_1_link: geometry collision mesh filename=meshes/spherical_wrist_1_link.STL; visual mesh filename=meshes/spherical_wrist_1_link.STL
- link spherical_wrist_2_link: geometry collision mesh filename=meshes/spherical_wrist_2_link.STL; visual mesh filename=meshes/spherical_wrist_2_link.STL
- link waiter_tray_link: geometry collision mesh filename=meshes/plate_shifted_scaled_origin_v3.STL; visual mesh filename=meshes/plate_shifted_scaled_origin_v3.STL

Commit message: edit end effector online + visualization script

File: Robots/kinova-gen3/kinova_grasp.urdf (robot description, URDF)
Before this commit: robot gen3_robotiq_2f_85, 11 links, 10 joints
Links:
- link base: geometry collision mesh filename=meshes/base_link.stl; visual mesh filename=meshes/base_link.stl
- link bracelet_link: geometry collision mesh filename=meshes/bracelet_with_vision_link.stl; visual mesh filename=meshes/bracelet_with_vision_link.stl
- link cube_link: geometry collision mesh filename=meshes/cup_hardware_shifted_scaled_rotated.stl; visual mesh filename=meshes/cup_hardware_shifted_scaled_rotated.stl
- link forearm_link: geometry collision mesh filename=meshes/forearm_link.stl; visual mesh filename=meshes/forearm_link.stl
- link gripper_base: geometry collision mesh filename=meshes/base_of_gripper.stl; visual mesh filename=meshes/base_of_gripper.stl
- link half_arm_1_link: geometry collision mesh filename=meshes/half_arm_1_link.stl; visual mesh filename=meshes/half_arm_1_link.stl
- link half_arm_2_link: geometry collision mesh filename=meshes/half_arm_2_link.stl; visual mesh filename=meshes/half_arm_2_link.stl
- link shoulder_link: geometry collision mesh filename=meshes/shoulder_link.stl; visual mesh filename=meshes/shoulder_link.stl
- link spherical_wrist_1_link: geometry collision mesh filename=meshes/spherical_wrist_1_link.stl; visual mesh filename=meshes/spherical_wrist_1_link.stl
- link spherical_wrist_2_link: geometry collision mesh filename=meshes/spherical_wrist_2_link.stl; visual mesh filename=meshes/spherical_wrist_2_link.stl
- link waiter_tray_link: geometry collision mesh filename=meshes/plate_shifted_scaled_origin_v3.stl; visual mesh filename=meshes/plate_shifted_scaled_origin_v3.stl
Joints:
- joint waiter_tray_joint: limit (none) -> effort=10000 velocity=10000; type fixed -> revolute

Commit message: change PZsparse reduce strategy

File: Robots/kinova-gen3/kinova_grasp.urdf (robot description, URDF)
Before this commit: robot gen3_robotiq_2f_85, 11 links, 10 joints
Links:
- link bracelet_link: mass 0.5 -> 0.5006
Joints:
- joint waiter_tray_joint: type revolute -> fixed
