Commit message: update kinova urdf with gripper

File: Robots/kinova-gen3/kinova_grasp_object.urdf (robot description, URDF)
Before this commit: robot gen3_robotiq_2f_85, 20 links, 19 joints
Links:
- link object_link: mass 2.0 -> 0.9072; geometry collision mesh filename=meshes/dumbbell_2lb.STL scale=0.001 0.001 0.001; visual mesh filename=meshes/dumbbell_2lb.STL scale=0.001 0.001 0.001
Joints:
- joint contact_joint: origin xyz=0 0 -0.171525 rpy=0 0 0 -> xyz=0 -0.16 0 rpy=0 1.5708 0
