Commit message: update dual arm Armour example

File: Robots/kinova-gen3/gen3_2f85.urdf (robot description, URDF)
Before this commit: robot gen3_, 21 links, 20 joints
Joints:
- removed joint gen3_joint_1
- removed joint gen3_joint_2
- removed joint gen3_joint_3
- removed joint gen3_joint_4
- removed joint gen3_joint_5
- removed joint gen3_joint_6
- removed joint gen3_joint_7
- added joint joint_1: type revolute, parent gen3_base_link, child gen3_shoulder_link, origin xyz=0 0 0.15643 rpy=3.1416 2.7629E-18 -4.9305E-36, axis 0 0 1, limit effort=39 velocity=1.3963
- added joint joint_2: type revolute, parent gen3_shoulder_link, child gen3_half_arm_1_link, origin xyz=0 0.005375 -0.12838 rpy=1.5708 2.1343E-17 -1.1102E-16, axis 0 0 1, limit lower=-2.41 upper=2.41 effort=39 velocity=1.3963
- added joint joint_3: type revolute, parent gen3_half_arm_1_link, child gen3_half_arm_2_link, origin xyz=0 -0.21038 -0.006375 rpy=-1.5708 1.2326E-32 -2.9122E-16, axis 0 0 1, limit effort=39 velocity=1.3963
- added joint joint_4: type revolute, parent gen3_half_arm_2_link, child gen3_forearm_link, origin xyz=0 0.006375 -0.21038 rpy=1.5708 -6.6954E-17 -1.6653E-16, axis 0 0 1, limit lower=-2.66 upper=2.66 effort=39 velocity=1.3963
- added joint joint_5: type revolute, parent gen3_forearm_link, child gen3_spherical_wrist_1_link, origin xyz=0 -0.20843 -0.006375 rpy=-1.5708 2.2204E-16 -6.373E-17, axis 0 0 1, limit effort=9 velocity=1.2218
- added joint joint_6: type revolute, parent gen3_spherical_wrist_1_link, child gen3_spherical_wrist_2_link, origin xyz=0 0.00017505 -0.10593 rpy=1.5708 9.2076E-28 -8.2157E-15, axis 0 0 1, limit lower=-2.23 upper=2.23 effort=9 velocity=1.2218
- added joint joint_7: type revolute, parent gen3_spherical_wrist_2_link, child gen3_bracelet_link, origin xyz=0 -0.10593 -0.00017505 rpy=-1.5708 -5.5511E-17 9.6396E-17, axis 0 0 1, limit effort=9 velocity=1.2218

File: Robots/kinova-gen3/gen3_2f85_fixed_object.urdf (robot description, URDF)
Before this commit: robot gen3_, 22 links, 21 joints
Joints:
- removed joint gen3_joint_1
- removed joint gen3_joint_2
- removed joint gen3_joint_3
- removed joint gen3_joint_4
- removed joint gen3_joint_5
- removed joint gen3_joint_6
- removed joint gen3_joint_7
- added joint joint_1: type revolute, parent gen3_base_link, child gen3_shoulder_link, origin xyz=0 0 0.15643 rpy=3.1416 2.7629E-18 -4.9305E-36, axis 0 0 1, limit effort=39 velocity=1.3963
- added joint joint_2: type revolute, parent gen3_shoulder_link, child gen3_half_arm_1_link, origin xyz=0 0.005375 -0.12838 rpy=1.5708 2.1343E-17 -1.1102E-16, axis 0 0 1, limit lower=-2.41 upper=2.41 effort=39 velocity=1.3963
- added joint joint_3: type revolute, parent gen3_half_arm_1_link, child gen3_half_arm_2_link, origin xyz=0 -0.21038 -0.006375 rpy=-1.5708 1.2326E-32 -2.9122E-16, axis 0 0 1, limit effort=39 velocity=1.3963
- added joint joint_4: type revolute, parent gen3_half_arm_2_link, child gen3_forearm_link, origin xyz=0 0.006375 -0.21038 rpy=1.5708 -6.6954E-17 -1.6653E-16, axis 0 0 1, limit lower=-2.66 upper=2.66 effort=39 velocity=1.3963
- added joint joint_5: type revolute, parent gen3_forearm_link, child gen3_spherical_wrist_1_link, origin xyz=0 -0.20843 -0.006375 rpy=-1.5708 2.2204E-16 -6.373E-17, axis 0 0 1, limit effort=9 velocity=1.2218
- added joint joint_6: type revolute, parent gen3_spherical_wrist_1_link, child gen3_spherical_wrist_2_link, origin xyz=0 0.00017505 -0.10593 rpy=1.5708 9.2076E-28 -8.2157E-15, axis 0 0 1, limit lower=-2.23 upper=2.23 effort=9 velocity=1.2218
- added joint joint_7: type revolute, parent gen3_spherical_wrist_2_link, child gen3_bracelet_link, origin xyz=0 -0.10593 -0.00017505 rpy=-1.5708 -5.5511E-17 9.6396E-17, axis 0 0 1, limit effort=9 velocity=1.2218

File: Robots/kinova-gen3/gen3_2f85_fixed_the_other_side.urdf (robot description, URDF)
Before this commit: robot gen3_2f85_fixed, 21 links, 20 joints
Joints:
- joint gen3_base_joint: origin xyz=0 0 0 rpy=0 0 0 -> xyz=1.36 0 0 rpy=0 0 3.1415926
