Commit message: add kinova longer horizon planner python script

File: Robots/kinova-gen3/gen3_2f85_fixed_object.urdf (robot description, URDF)
Before this commit: robot gen3_2f85_fixed_object, 22 links, 21 joints
Links:
- link object_link: mass 0.9072 -> 2.72155422; geometry collision mesh filename=meshes/dumbbell_6lb.STL scale=0.001 0.001 0.001; visual mesh filename=meshes/dumbbell_6lb.STL scale=0.001 0.001 0.001
