Commit message: update kinova urdf

File: Robots/kinova-gen3/kinova_suction_plate.urdf (robot description, URDF)
Before this commit: robot gen3_robotiq_2f_85, 9 links, 8 joints
Links:
- link base: geometry collision mesh filename=meshes/base_link.stl; visual mesh filename=meshes/base_link.stl
- link composite_link: geometry collision mesh filename=meshes/bracelet_with_vision_link.stl; visual mesh filename=meshes/bracelet_with_vision_link.stl
- link forearm_link: geometry collision mesh filename=meshes/forearm_link.stl; visual mesh filename=meshes/forearm_link.stl
- link half_arm_1_link: geometry collision mesh filename=meshes/half_arm_1_link.stl; visual mesh filename=meshes/half_arm_1_link.stl
- link half_arm_2_link: geometry collision mesh filename=meshes/half_arm_2_link.stl; visual mesh filename=meshes/half_arm_2_link.stl
- link object_link: geometry collision mesh filename=meshes/suction_plate_v2.stl; visual mesh filename=meshes/suction_plate_v2.stl
- link shoulder_link: geometry collision mesh filename=meshes/shoulder_link.stl; visual mesh filename=meshes/shoulder_link.stl
- link spherical_wrist_1_link: geometry collision mesh filename=meshes/spherical_wrist_1_link.stl; visual mesh filename=meshes/spherical_wrist_1_link.stl
- link spherical_wrist_2_link: geometry collision mesh filename=meshes/spherical_wrist_2_link.stl; visual mesh filename=meshes/spherical_wrist_2_link.stl
Joints:
- joint contact_joint: origin xyz=0 0 -0.171525 rpy=0 0 0 -> xyz=0 0 -0.125 rpy=0 0 0
