Commit message: update optimizer for multiple calls on one instance

File: Robots/kinova-gen3/kinova.urdf (robot description, URDF)
Before this commit: robot gen3, 9 links, 8 joints
Links:
- link base_link: geometry collision mesh filename=meshes/base_link.stl; visual mesh filename=meshes/base_link.stl
- link bracelet_link: geometry collision mesh filename=meshes/bracelet_no_vision_link.stl; visual mesh filename=meshes/bracelet_no_vision_link.stl
- link end_effector_link: geometry 
- link forearm_link: geometry collision mesh filename=meshes/forearm_link.stl; visual mesh filename=meshes/forearm_link.stl
- link half_arm_1_link: geometry collision mesh filename=meshes/half_arm_1_link.stl; visual mesh filename=meshes/half_arm_1_link.stl
- link half_arm_2_link: geometry collision mesh filename=meshes/half_arm_2_link.stl; visual mesh filename=meshes/half_arm_2_link.stl
- link shoulder_link: geometry collision mesh filename=meshes/shoulder_link.stl; visual mesh filename=meshes/shoulder_link.stl
- link spherical_wrist_1_link: geometry collision mesh filename=meshes/spherical_wrist_1_link.stl; visual mesh filename=meshes/spherical_wrist_1_link.stl
- link spherical_wrist_2_link: geometry collision mesh filename=meshes/spherical_wrist_2_link.stl; visual mesh filename=meshes/spherical_wrist_2_link.stl

Commit message: 1

File: Robots/kinova-gen3/kinova.urdf (robot description, URDF)
Before this commit: robot gen3, 9 links, 8 joints
Links:
- link base_link: geometry collision mesh filename=meshes/base_link.stl; visual mesh filename=meshes/base_link.stl
- link bracelet_link: geometry collision mesh filename=meshes/bracelet_no_vision_link.stl; visual mesh filename=meshes/bracelet_no_vision_link.stl
- link forearm_link: geometry collision mesh filename=meshes/forearm_link.stl; visual mesh filename=meshes/forearm_link.stl
- link half_arm_1_link: geometry collision mesh filename=meshes/half_arm_1_link.stl; visual mesh filename=meshes/half_arm_1_link.stl
- link half_arm_2_link: geometry collision mesh filename=meshes/half_arm_2_link.stl; visual mesh filename=meshes/half_arm_2_link.stl
- link shoulder_link: geometry collision mesh filename=meshes/shoulder_link.stl; visual mesh filename=meshes/shoulder_link.stl
- link spherical_wrist_1_link: geometry collision mesh filename=meshes/spherical_wrist_1_link.stl; visual mesh filename=meshes/spherical_wrist_1_link.stl
- link spherical_wrist_2_link: geometry collision mesh filename=meshes/spherical_wrist_2_link.stl; visual mesh filename=meshes/spherical_wrist_2_link.stl

Commit message: another way to compute torque reachsets using rnea

File: Robots/kinova-gen3/kinova.urdf (robot description, URDF)
Before this commit: robot GEN3-7DOF-VISION_ARM_URDF_V12, 12 links, 11 joints
Links:
- removed link camera_color_frame
- removed link camera_depth_frame
- removed link camera_link
Joints:
- removed joint camera_module
- removed joint color_module
- removed joint depth_module
