Commit message: bugfix in DynamicsConstraints in walking robots + fix arm positions for G1

File: Robots/unitree-g1/g1_22dof.urdf (robot description, URDF)
Before this commit: robot g1_12dof_floatingbase, 39 links, 38 joints
Links:
- removed link Px
- removed link Py
- removed link Pz
- removed link Rx
- removed link Ry
- removed link ground
Joints:
- removed joint Px_joint
- removed joint Py_joint
- removed joint Pz_joint
- removed joint Rx_joint
- removed joint Ry_joint
- removed joint Rz_joint
- joint left_elbow_joint: type fixed -> revolute
- joint left_shoulder_pitch_joint: type fixed -> revolute
- joint left_shoulder_roll_joint: type fixed -> revolute
- joint left_shoulder_yaw_joint: type fixed -> revolute
- joint left_wrist_roll_joint: type fixed -> revolute
- joint right_elbow_joint: type fixed -> revolute
- joint right_shoulder_pitch_joint: type fixed -> revolute
- joint right_shoulder_roll_joint: type fixed -> revolute
- joint right_shoulder_yaw_joint: type fixed -> revolute
- joint right_wrist_roll_joint: type fixed -> revolute

File: Robots/unitree-g1/g1_22dof_floatingbase.urdf (robot description, URDF)
Before this commit: robot g1_12dof_floatingbase, 39 links, 38 joints
Joints:
- joint left_elbow_joint: type fixed -> revolute
- joint left_shoulder_pitch_joint: type fixed -> revolute
- joint left_shoulder_roll_joint: type fixed -> revolute
- joint left_shoulder_yaw_joint: type fixed -> revolute
- joint left_wrist_roll_joint: type fixed -> revolute
- joint right_elbow_joint: type fixed -> revolute
- joint right_shoulder_pitch_joint: type fixed -> revolute
- joint right_shoulder_roll_joint: type fixed -> revolute
- joint right_shoulder_yaw_joint: type fixed -> revolute
- joint right_wrist_roll_joint: type fixed -> revolute
